Commit message: Update tibia joint range

File: simulate/robot/SpiderBot.urdf (robot description, URDF)
Before this commit: robot SpiderBody, 97 links, 96 joints
Joints:
- joint Leg1_Tibia: limit lower=0.4 upper=2.7 effort=1000000 velocity=1000000 -> lower=0.0 upper=2.7 effort=1000000 velocity=1000000
- joint Leg2_Tibia: limit lower=0.4 upper=2.7 effort=1000000 velocity=1000000 -> lower=0.0 upper=2.7 effort=1000000 velocity=1000000
- joint Leg3_Tibia: limit lower=0.4 upper=2.7 effort=1000000 velocity=1000000 -> lower=0.0 upper=2.7 effort=1000000 velocity=1000000
- joint Leg4_Tibia: limit lower=0.4 upper=2.7 effort=1000000 velocity=1000000 -> lower=0.0 upper=2.7 effort=1000000 velocity=1000000
- joint Leg5_Tibia: limit lower=0.4 upper=2.7 effort=1000000 velocity=1000000 -> lower=0.0 upper=2.7 effort=1000000 velocity=1000000
- joint Leg6_Tibia: limit lower=0.4 upper=2.7 effort=1000000 velocity=1000000 -> lower=0.0 upper=2.7 effort=1000000 velocity=1000000
- joint Leg7_Tibia: limit lower=0.4 upper=2.7 effort=1000000 velocity=1000000 -> lower=0.0 upper=2.7 effort=1000000 velocity=1000000
- joint Leg8_Tibia: limit lower=0.4 upper=2.7 effort=1000000 velocity=1000000 -> lower=0.0 upper=2.7 effort=1000000 velocity=1000000

Commit message: Fix joint USD APIs, so they move in issac sim

File: simulate/robot/SpiderBot.urdf (robot description, URDF)
Before this commit: robot SpiderBody, 97 links, 96 joints
Joints:
- joint Leg1_Tibia: limit lower=0.0 upper=2.7 effort=1000000 velocity=1000000 -> lower=-2.7 upper=0.0 effort=1000000 velocity=1000000
- joint Leg2_Tibia: limit lower=0.0 upper=2.7 effort=1000000 velocity=1000000 -> lower=-2.7 upper=0.0 effort=1000000 velocity=1000000
- joint Leg3_Tibia: limit lower=0.0 upper=2.7 effort=1000000 velocity=1000000 -> lower=-2.7 upper=0.0 effort=1000000 velocity=1000000
- joint Leg4_Tibia: limit lower=0.0 upper=2.7 effort=1000000 velocity=1000000 -> lower=-2.7 upper=0.0 effort=1000000 velocity=1000000
- joint Leg5_Tibia: limit lower=0.0 upper=2.7 effort=1000000 velocity=1000000 -> lower=-2.7 upper=0.0 effort=1000000 velocity=1000000
- joint Leg6_Tibia: limit lower=0.0 upper=2.7 effort=1000000 velocity=1000000 -> lower=-2.7 upper=0.0 effort=1000000 velocity=1000000
- joint Leg7_Tibia: limit lower=0.0 upper=2.7 effort=1000000 velocity=1000000 -> lower=-2.7 upper=0.0 effort=1000000 velocity=1000000
- joint Leg8_Tibia: limit lower=0.0 upper=2.7 effort=1000000 velocity=1000000 -> lower=-2.7 upper=0.0 effort=1000000 velocity=1000000

Commit message: Cleanup model and rewards for standing

File: simulate/robot/SpiderBot.urdf (robot description, URDF)
Before this commit: robot SpiderBody, 97 links, 96 joints
Joints:
- joint Leg1_Tibia: limit lower=-2.7 upper=0.0 effort=1000000 velocity=1000000 -> lower=0.0 upper=2.7 effort=1000000 velocity=1000000
- joint Leg2_Tibia: limit lower=-2.7 upper=0.0 effort=1000000 velocity=1000000 -> lower=0.0 upper=2.7 effort=1000000 velocity=1000000
- joint Leg3_Tibia: limit lower=-2.7 upper=0.0 effort=1000000 velocity=1000000 -> lower=0.0 upper=2.7 effort=1000000 velocity=1000000
- joint Leg4_Tibia: limit lower=-2.7 upper=0.0 effort=1000000 velocity=1000000 -> lower=0.0 upper=2.7 effort=1000000 velocity=1000000
- joint Leg5_Tibia: limit lower=-2.7 upper=0.0 effort=1000000 velocity=1000000 -> lower=0.0 upper=2.7 effort=1000000 velocity=1000000
- joint Leg6_Tibia: limit lower=-2.7 upper=0.0 effort=1000000 velocity=1000000 -> lower=0.0 upper=2.7 effort=1000000 velocity=1000000
- joint Leg7_Tibia: limit lower=-2.7 upper=0.0 effort=1000000 velocity=1000000 -> lower=0.0 upper=2.7 effort=1000000 velocity=1000000
- joint Leg8_Tibia: limit lower=-2.7 upper=0.0 effort=1000000 velocity=1000000 -> lower=0.0 upper=2.7 effort=1000000 velocity=1000000
